Commit message: nav update

File: my_robot_controller/urdf/simple_robot.urdf (robot description, URDF)
Before this commit: robot simple_robot, 11 links, 10 joints
Links:
- removed link led_back_left_link
- removed link led_back_right_link
- removed link led_front_left_link
- removed link led_front_right_link
- removed link wheel_left_back_link
- removed link wheel_right_back_link
- added link imu_link; visual box size=0.02 0.02 0.01
- link wheel_left_link: mass None -> 0.5; geometry collision cylinder length=0.05 radius=0.1; visual cylinder length=0.05 radius=0.1
- link wheel_right_link: mass None -> 0.5; geometry collision cylinder length=0.05 radius=0.1; visual cylinder length=0.05 radius=0.1
Joints:
- removed joint base_to_led_back_left
- removed joint base_to_led_back_right
- removed joint base_to_led_front_left
- removed joint base_to_led_front_right
- removed joint base_to_left_back_wheel
- removed joint base_to_right_back_wheel
- added joint base_to_imu: type fixed, parent base_link, child imu_link, origin xyz=0 0 0.055 rpy=0 0 0
- joint base_to_left_wheel: origin xyz=0.15 0.175 0 rpy=1.5708 0 0 -> xyz=0 0.175 0 rpy=1.5708 0 0
- joint base_to_right_wheel: origin xyz=0.15 -0.175 0 rpy=1.5708 0 0 -> xyz=0 -0.175 0 rpy=1.5708 0 0
